File: board/beeb.kicad_pcb (KiCad board)
At the start: 2 copper layers, 76.2 x 53.3 mm, 36 parts, among them J2 AVR-JTAG-10, SW1 SW_DIP_x08, U1 WIT122UH, U2 ps2, U3 XC95144XL-TQ100, U4 beebKB, U5 LM1117-3.3

Commit message: Update silkscreen
Other:
- board text added: "DISK/~NET~"
- board text added: "GND TDI GND VCC GND TMS VREF TDO GND TCK"
- board text removed: "DISK/NET"
- board text removed: "GND TDI GND +5v GND TMS GND TDO GND TCK"
Changed lines of the file:
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@@
   (layers
     (0 F.Cu signal)
-    (31 B.Cu signal)
+    (31 B.Cu signal hide)
     (32 B.Adhes user)
     (33 F.Adhes user)
@@
   (gr_line (start 52.07 108.585) (end 52.07 113.665) (layer F.SilkS) (width 0.12))
   (gr_line (start 48.26 108.585) (end 52.07 108.585) (layer F.SilkS) (width 0.12))
-  (gr_text "GND TDI\nGND +5v\nGND TMS\nGND TDO\nGND TCK" (at 50.165 111.125) (layer F.SilkS)
+  (gr_text "GND TDI\nGND VCC\nGND TMS\nVREF TDO\nGND TCK" (at 50.165 111.125) (layer F.SilkS)
     (effects (font (size 0.5 0.5) (thickness 0.125)))
   )
@@
   (gr_line (start 57.15 102.87) (end 59.69 102.87) (layer F.SilkS) (width 0.12))
   (gr_line (start 57.15 90.805) (end 57.15 102.87) (layer F.SilkS) (width 0.12))
-  (gr_text DISK/NET (at 58.42 96.52 90) (layer F.SilkS)
+  (gr_text DISK/~NET~ (at 58.42 96.52 90) (layer F.SilkS)
     (effects (font (size 1 1) (thickness 0.25)))
   )

Commit message: Make it work
Parts:
- added R14: R, Resistor_SMD:R_1206_3216Metric_Pad1.42x1.75mm_HandSolder, F.Cu at (51.3, 110.5)
- added R15: R, Resistor_SMD:R_1206_3216Metric_Pad1.42x1.75mm_HandSolder, F.Cu at (56.5, 110.5)
- added R16: 10K, Resistor_SMD:R_1206_3216Metric_Pad1.42x1.75mm_HandSolder, F.Cu at (55.4, 96.6)
- added R17: R_Small, Resistor_SMD:R_1206_3216Metric_Pad1.42x1.75mm_HandSolder, B.Cu at (58.4, 85.1)
- added R18: R_Small, Resistor_SMD:R_1206_3216Metric_Pad1.42x1.75mm_HandSolder, B.Cu at (61.0, 85.1)
- added R19: R_Small, Resistor_SMD:R_1206_3216Metric_Pad1.42x1.75mm_HandSolder, B.Cu at (63.5, 85.1)
- added R20: R_Small, Resistor_SMD:R_1206_3216Metric_Pad1.42x1.75mm_HandSolder, B.Cu at (66.0, 85.1)
- added R21: R_Small, Resistor_SMD:R_1206_3216Metric_Pad1.42x1.75mm_HandSolder, B.Cu at (68.6, 85.1)
- added R22: R_Small, Resistor_SMD:R_1206_3216Metric_Pad1.42x1.75mm_HandSolder, B.Cu at (71.1, 85.1)
- added R23: R_Small, Resistor_SMD:R_1206_3216Metric_Pad1.42x1.75mm_HandSolder, B.Cu at (73.7, 85.1)
- added R24: R_Small, Resistor_SMD:R_1206_3216Metric_Pad1.42x1.75mm_HandSolder, B.Cu at (76.2, 85.1)
- added R25: 10K, Resistor_SMD:R_1206_3216Metric_Pad1.42x1.75mm_HandSolder, F.Cu at (102.9, 94.6)
- added R26: 10K, Resistor_SMD:R_1206_3216Metric_Pad1.42x1.75mm_HandSolder, F.Cu at (106.0, 94.6)
- added RV1: R_POT, Potentiometer_THT:Potentiometer_Bourns_3386C_Horizontal, F.Cu at (62.2, 106.0)
- added TP1: TP_PWROK, Connector_PinHeader_2.54mm:PinHeader_1x01_P2.54mm_Vertical, F.Cu at (90.8, 122.6)
- added U6: 74LS244_Split, Package_SO:SOIC-20W_7.5x12.8mm_P1.27mm, F.Cu at (62.9, 120.2)
- added U7: 74LS244_Split, Package_SO:SOIC-20W_7.5x12.8mm_P1.27mm, F.Cu at (99.7, 120.0)
- added U8: LM2903, Package_SO:SOP-8_5.28x5.23mm_P1.27mm, F.Cu at (53.1, 105.2)
- C3: moved to B.Cu
- U5: footprint Package_TO_SOT_THT:TO-220-3_Horizontal_TabDown -> Package_TO_SOT_SMD:SOT-223-3_TabPin2
- moved R12 17.1 mm to (103.6, 105.4), turned to 0 degrees
- moved R11 14.1 mm to (103.6, 108.0), turned to 0 degrees
- moved R13 11.4 mm to (103.6, 110.5), turned to 0 degrees
- moved U5 9.03 mm to (51.4, 118.1), turned to 90 degrees
- moved LEDS1 7.41 mm to (99.1, 110.5)
- moved C3 6.38 mm to (87.6, 114.3), turned to 90 degrees
- moved C7 6.13 mm to (87.0, 99.4), turned to 90 degrees
- moved J2 4.44 mm to (51.4, 99.1)
- moved RESET1 4.02 mm to (99.1, 101.6), turned to 180 degrees
- moved U1 1.59 mm to (97.0, 97.0)
- moved C4 1.27 mm to (82.5, 123.8)
- moved C6 1.08 mm to (73.0, 104.1), turned to 180 degrees
- moved SW1 0.25 mm to (76.2, 81.0)
Connections:
- C4 pad 1: +5V -> +3V3
- C5 pad 1: +5V -> +3V3
- C6 pad 1: +5V -> +3V3
- C7 pad 1: +5V -> +3V3
- R11 pad 1: Net-(LEDS1-Pad1) -> Net-(LEDS1-Pad3)
- R12 pad 1: Net-(LEDS1-Pad3) -> Net-(LEDS1-Pad5)
- R13 pad 1: Net-(LEDS1-Pad5) -> Net-(LEDS1-Pad1)
- U3 pad 12: /W -> /W_BUF
- U3 pad 13: (no net) -> /W_EN
- U3 pad 22: /BEEBCLK -> /BEEBCLK_BUF
- U3 pad 81: /CB -> /CB_BUF
- U3 pad 82: /COL0 -> /COL0_BUF
- U3 pad 85: /COL1 -> /COL1_BUF
- U3 pad 86: /COL2 -> /COL2_BUF
- U3 pad 87: (no net) -> /ROW3_BUF
- U3 pad 89: /ROW0 -> /ROW0_BUF
- U3 pad 90: /ROW1 -> /ROW1_BUF
- U3 pad 91: /ROW2 -> /ROW2_BUF
- U4 pad 11: (no net) -> /ROW3
Routing:
- net +3V3: track 121.6 -> 233.7 mm, vias 5 -> 6
- net /PWROK: track 0.00 -> 98.2 mm, vias 0 -> 3
- net +5V: track 148.2 -> 241.3 mm, vias 6 -> 1
- net GND: track 43.4 -> 87.4 mm, vias 15 -> 16
- net /BEEBCLK_BUF: track 0.00 -> 36.4 mm, vias 0 -> 2
- net /CB_BUF: track 0.00 -> 34.1 mm, vias 0 -> 2
- net /COL2_BUF: track 0.00 -> 33.3 mm
- net /ROW3_BUF: track 0.00 -> 32.9 mm
- net /ROW3: track 0.00 -> 30.5 mm, vias 0 -> 1
- net /ROW1_BUF: track 0.00 -> 29.9 mm
- net /ROW2_BUF: track 0.00 -> 28.8 mm
- net Net-(RESET1-Pad2): track 55.8 -> 83.9 mm
- net /ROW0_BUF: track 0.00 -> 26.5 mm
- net /BEEBCLK: track 36.6 -> 10.6 mm
- net /COL1_BUF: track 0.00 -> 25.8 mm
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- removed copper zone on F.Cu, net GND
Other:
- board text added: "CAPS"
- board text added: "CAS"
- board text added: "LEDs"
- board text added: "NO HOT- PLUG"
- board text added: "RESET"
- board text added: "SHFT"
- board text removed: "GND TDI GND VCC GND TMS VREF TDO GND TCK"
